Commit message: Debuget CtrlAviary

File: RRT_gym_pybullet_combination/obstacles/box2.urdf (robot description, URDF)
Before this commit: robot test.urdf, 1 links, 0 joints
Links:
- link baseLink: mass .1 -> 0; geometry visual box size=5 5 5

Commit message: Load all .urdf files from the folder obstacles

File: RRT_gym_pybullet_combination/obstacles/box2.urdf (robot description, URDF)
Before this commit: robot test.urdf, 1 links, 0 joints
Links:
- link baseLink: geometry visual box size=1 1 1
